File: Konami Justifier SFC/KiCad/Konami Justifier Main/Konami Justifier Main.kicad_sch (KiCad schematic)
At the start: 18 parts, among them J1 RJ12, J3 Conn_01x06_Socket, U1 74VHC9164FT

Commit message: Add files via upload
Parts:
- removed MD-R1: 93 Ohm 1%, Resistor_THT:R_Axial_DIN0207_L6.3mm_D2.5mm_P10.16mm_Horizontal, symbol Device:R
- added MD-C1: 100nF, Capacitor_THT:C_Axial_L3.8mm_D2.6mm_P10.00mm_Horizontal, symbol Device:C
Connections:
- net +5V: now also MD-C1.1
- net GND: now also MD-C1.2
Other:
- moved on the sheet: SFC-C1

Commit message: Add files via upload
Parts:
- removed MD-C1: 100nF, Capacitor_THT:C_Axial_L3.8mm_D2.6mm_P10.00mm_Horizontal, symbol Device:C
- removed SFC-C1: 100nF, Capacitor_THT:C_Disc_D5.0mm_W2.5mm_P5.00mm, symbol Device:C
- added C2: 100nF, Capacitor_THT:C_Disc_D5.0mm_W2.5mm_P5.00mm, symbol Device:C
- renumbered J3 to J2, MD-R2 to MD-R1, SFC-C2 to SFC-C1, SFC-R3 to SFC-R1
Connections:
- net +5V: now also C1.2, C2.1; no longer C1.1
- net GND: now also C1.1, C2.2; no longer C1.2
Other:
- moved on the sheet: C1

Commit message: Add files via upload
Parts:
- J1: footprint Connector_RJ:RJ12_Amphenol_54601-x06_Horizontal -> Connector_RJ:RJ25_Wayconn_MJEA-660X1_Horizontal
Changed lines of the file:
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@@
 			)
 		)
-		(property "Footprint" "Connector_RJ:RJ12_Amphenol_54601-x06_Horizontal"
+		(property "Footprint" "Connector_RJ:RJ25_Wayconn_MJEA-660X1_Horizontal"
 			(at 60.96 149.225 90)
 			(effects

Commit message: Add files via upload
Parts:
- removed SFC1: Conn_01x05_Pin, Connector_Molex:Molex_SL_171971-0005_1x05_P2.54mm_Vertical, symbol Connector:Conn_01x05_Pin
- removed SFC2: Conn_01x01_Pin, Connector_Pin:Pin_D1.0mm_L10.0mm_LooseFit, symbol Connector:Conn_01x01_Pin
- added SFC1: Conn_01x08_Pin, Connector_Molex:Molex_SL_171971-0008_1x08_P2.54mm_Vertical, symbol Connector:Conn_01x08_Pin
Connections:
- net +5V: now also SFC1.8 (Pin_8)
- net GND: now also SFC1.1 (Pin_1)
- net at SFC-TP1.1, U1.10 (Q/D5): now also SFC1.2 (Pin_2)
- net at MD1.3 (Pin_3), SFC-C1.1, U1.9 (Q/D4): now also SFC1.3 (Pin_3)
- net at MD1.5 (Pin_5), SFC-TP2.1, U1.5 (Q/D1): now also SFC1.4 (Pin_4)
- net at MD1.6 (Pin_6), SFC-TP6.1, U1.6 (Q/D2): now also SFC1.5 (Pin_5)
- no-connect marks 0 -> 2
