File: Konami Justifier SFC/KiCad/Konami Justifier Main/Konami Justifier Main.kicad_pcb (KiCad board)
At the start: 4 copper layers, 25.2 x 50 mm, 21 parts, among them J1 RJ12, J3 Conn_01x06_Socket, U1 74VHC9164FT

Commit message: Add files via upload
Parts:
- removed MD-R1: 93 Ohm 1%, Resistor_THT:R_Axial_DIN0207_L6.3mm_D2.5mm_P10.16mm_Horizontal
- added MD-C1: 100nF, Capacitor_THT:C_Axial_L3.8mm_D2.6mm_P10.00mm_Horizontal, F.Cu at (145.3, 78.5)
Changed lines of the file:
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@@
 		(property ki_fp_filters "Pin* Test*")
 		(sheetname "/")
-		(sheetfile "Konami Justifier 02.kicad_sch")
+		(sheetfile "Konami Justifier Main.kicad_sch")
 		(attr exclude_from_pos_files)
 		(fp_circle
@@
 		(property ki_fp_filters "Pin* Test*")
 		(sheetname "/")
-		(sheetfile "Konami Justifier 02.kicad_sch")
+		(sheetfile "Konami Justifier Main.kicad_sch")
 		(attr exclude_from_pos_files)
 		(fp_circle
@@
 		(property ki_fp_filters "6P6C* RJ12* RJ18* RJ25*")
 		(sheetname "/")
-		(sheetfile "Konami Justifier 02.kicad_sch")
+		(sheetfile "Konami Justifier Main.kicad_sch")
 		(attr through_hole)
 		(fp_line
@@
 		(embedded_fonts no)
 	)
-	(footprint "Resistor_THT:R_Axial_DIN0207_L6.3mm_D2.5mm_P10.16mm_Horizontal"
-		(layer "F.Cu")
-		(at 145.34 78.5)
-		(descr "Resistor, Axial_DIN0207 series, Axial, Horizontal, pin pitch=10.16mm, 0.25W = 1/4W, length*diameter=6.3*2.5mm^2, http://cdn-reichelt.de/documents/datenblatt/B400/1_4W%23YAG.pdf")
-		(tags "Resistor Axial_DIN0207 series Axial Horizontal pin pitch 10.16mm 0.25W = 1/4W length 6.3mm diameter 2.5mm")
-		(property "Reference" "MD-R1"
-			(at 5.08 0 0)
-			(layer "F.SilkS")
-			(effects
-				(font
-					(size 1 1)
-					(thickness 0.15)
-				)
-			)
-		)
-		(property "Value" "93 Ohm 1%"
-			(at 5.08 2.37 0)
-			(layer "F.Fab")
-			(effects
-				(font
-					(size 1 1)
-					(thickness 0.15)
-				)
-			)
-		)
-		(property "Datasheet" "~"
-			(at 0 0 0)
-			(layer "F.Fab")
-			(hide yes)
-			(effects
-				(font
-					(size 1.27 1.27)
-					(thickness 0.15)
-				)
-			)
-		)
-		(property "Description" "Resistor"
-			(at 0 0 0)
-			(layer "F.Fab")
-			(hide yes)
-			(effects
-				(font
-					(size 1.27 1.27)
-					(thickness 0.15)
-				)
-			)
-		)
-		(property ki_fp_filters "R_*")
-		(sheetname "/")
-		(sheetfile "Konami Justifier 02.kicad_sch")
-		(attr through_hole)
-		(fp_line
-			(start 1.04 0)
-			(end 1.81 0)
-			(stroke
-				(width 0.12)
-				(type solid)
-			)
-			(layer "F.SilkS")
-		)
-		(fp_line
-			(start 9.12 0)
-			(end 8.35 0)
-			(stroke
-				(width 0.12)
-				(type solid)
-			)
-			(layer "F.SilkS")
-		)
-		(fp_rect
-			(start 1.81 -1.37)
-			(end 8.35 1.37)
-			(stroke
-				(width 0.12)
-				(type solid)
-			)
-			(fill no)
-			(layer "F.SilkS")
-		)
-		(fp_rect
-			(start -1.05 -1.5)
-			(end 11.21 1.5)
-			(stroke
-				(width 0.05)
-				(type solid)
-			)
-			(fill no)
-			(layer "F.CrtYd")
-		)
-		(fp_line
-			(start 0 0)
-			(end 1.93 0)
-			(stroke
-				(width 0.1)
-				(type solid)
-			)
-			(layer "F.Fab")
-		)
-		(fp_line
-			(start 10.16 0)
-			(end 8.23 0)
-			(stroke
-				(width 0.1)
-				(type solid)
-			)
-			(layer "F.Fab")
-		)
-		(fp_rect
-			(start 1.93 -1.25)
-			(end 8.23 1.25)
-			(stroke
-				(width 0.1)
-				(type solid)
-			)
-			(fill no)
-			(layer "F.Fab")
-		)
-		(fp_text user "${REFERENCE}"
-			(at 5.08 0 0)
-			(layer "F.Fab")
-			(effects
-				(font
-					(size 1 1)
-					(thickness 0.15)
-				)
-			)
-		)
-		(pad "1" thru_hole circle
-			(at 0 0)
-			(size 1.6 1.6)
-			(drill 0.8)
-			(layers "*.Cu" "*.Mask")
-			(remove_unused_layers no)
-			(net 6 "+5V")
-			(pintype "passive")
-		)
-		(pad "2" thru_hole circle
-			(at 10.16 0)
-			(size 1.6 1.6)
-			(drill 0.8)
-			(layers "*.Cu" "*.Mask")
-			(remove_unused_layers no)
-			(net 5 "GND")
-			(pintype "passive")
-		)
-		(embedded_fonts no)
-		(model "${KICAD9_3DMODEL_DIR}/Resistor_THT.3dshapes/R_Axial_DIN0207_L6.3mm_D2.5mm_P10.16mm_Horizontal.step"
-			(offset
-				(xyz 0 0 0)
-			)
-			(scale
-				(xyz 1 1 1)
-			)
-			(rotate
-				(xyz 0 0 0)
-			)
-		)
-	)
 	(footprint "Connector_Molex:Molex_SL_171971-0006_1x06_P2.54mm_Vertical"
 		(layer "F.Cu")
@@
 		(property ki_fp_filters "Connector*:*_1x??_*")
 		(sheetname "/")
-		(sheetfile "Konami Justifier 02.kicad_sch")
+		(sheetfile "Konami Justifier Main.kicad_sch")
 		(attr through_hole)
 		(fp_line
@@
 		(property ki_fp_filters "Pin* Test*")
 		(sheetname "/")
-		(sheetfile "Konami Justifier 02.kicad_sch")
+		(sheetfile "Konami Justifier Main.kicad_sch")
 		(attr exclude_from_pos_files)
 		(fp_circle
@@
 		(property ki_fp_filters "Connector*:*_1x??_*")
 		(sheetname "/")
-		(sheetfile "Konami Justifier 02.kicad_sch")
+		(sheetfile "Konami Justifier Main.kicad_sch")
 		(attr through_hole)
 		(fp_circle
@@
 		)
 	)
+	(footprint "Capacitor_THT:C_Axial_L3.8mm_D2.6mm_P10.00mm_Horizontal"
+		(layer "F.Cu")
+		(at 145.3 78.5)
+		(descr "C, Axial series, Axial, Horizontal, pin pitch=10mm, length*diameter=3.8*2.6mm^2, http://www.vishay.com/docs/45231/arseries.pdf")
+		(tags "C Axial series Axial Horizontal pin pitch 10mm  length 3.8mm diameter 2.6mm")
+		(property "Reference" "MD-C1"
+			(at 5 1.42 0)
+			(layer "F.SilkS")
+			(effects
+				(font
+					(size 1 1)
+					(thickness 0.15)
+				)
+			)
+		)
+		(property "Value" "100nF"
+			(at 5 2.42 0)
+			(layer "F.Fab")
+			(effects
+				(font
+					(size 1 1)
+					(thickness 0.15)
+				)
+			)
+		)
+		(property "Datasheet" "~"
+			(at 0 0 0)
+			(layer "F.Fab")
+			(hide yes)
+			(effects
+				(font
+					(size 1.27 1.27)
+					(thickness 0.15)
+				)
+			)
+		)
+		(property "Description" "Unpolarized capacitor"
+			(at 0 0 0)
+			(layer "F.Fab")
+			(hide yes)
+			(effects
+				(font
+					(size 1.27 1.27)
+					(thickness 0.15)
+				)
+			)
+		)
+		(property ki_fp_filters "C_*")
+		(sheetname "/")
+		(sheetfile "Konami Justifier Main.kicad_sch")
+		(attr through_hole)
+		(fp_line
+			(start 1.04 0)
+			(end 2.98 0)
+			(stroke
+				(width 0.12)
+				(type solid)
+			)
+			(layer "F.SilkS")
+		)
+		(fp_line
+			(start 8.96 0)
+			(end 7.02 0)
+			(stroke
+				(width 0.12)
+				(type solid)
+			)
+			(layer "F.SilkS")
+		)
+		(fp_rect
+			(start 2.98 -1.42)
+			(end 7.02 1.42)
+			(stroke
+				(width 0.12)
+				(type solid)
+			)
+			(fill no)
+			(layer "F.SilkS")
+		)
+		(fp_rect
+			(start -1.05 -1.55)
+			(end 11.05 1.55)
+			(stroke
+				(width 0.05)
+				(type solid)
+			)
+			(fill no)
+			(layer "F.CrtYd")
+		)
+		(fp_line
+			(start 0 0)
+			(end 3.1 0)
+			(stroke
+				(width 0.1)
+				(type solid)
+			)
+			(layer "F.Fab")
+		)
+		(fp_line
+			(start 10 0)
+			(end 6.9 0)
+			(stroke
+				(width 0.1)
+				(type solid)
+			)
+			(layer "F.Fab")
+		)
+		(fp_rect
+			(start 3.1 -1.3)
+			(end 6.9 1.3)
+			(stroke
+				(width 0.1)
+				(type solid)
+			)
+			(fill no)
+			(layer "F.Fab")
+		)
+		(fp_text user "${REFERENCE}"
+			(at 5 0 0)
+			(layer "F.Fab")
+			(effects
+				(font
+					(size 0.76 0.76)
+					(thickness 0.114)
+				)
+			)
+		)
+		(pad "1" thru_hole circle
+			(at 0 0)
+			(size 1.6 1.6)
+			(drill 0.8)
+			(layers "*.Cu" "*.Mask")
+			(remove_unused_layers no)
+			(net 6 "+5V")
+			(pintype "passive")
+		)
+		(pad "2" thru_hole circle
+			(at 10 0)
+			(size 1.6 1.6)
+			(drill 0.8)
+			(layers "*.Cu" "*.Mask")
+			(remove_unused_layers no)
+			(net 5 "GND")
+			(pintype "passive")
+		)
+		(embedded_fonts no)
+		(model "${KICAD9_3DMODEL_DIR}/Capacitor_THT.3dshapes/C_Axial_L3.8mm_D2.6mm_P10.00mm_Horizontal.step"
+			(offset
+				(xyz 0 0 0)
+			)
+			(scale
+				(xyz 1 1 1)
+			)
+			(rotate
+				(xyz 0 0 0)
+			)
+		)
+	)
 	(footprint "TestPoint:TestPoint_THTPad_D1.5mm_Drill0.7mm"
 		(layer "F.Cu")
@@
 		(property ki_fp_filters "Pin* Test*")
 		(sheetname "/")
-		(sheetfile "Konami Justifier 02.kicad_sch")
+		(sheetfile "Konami Justifier Main.kicad_sch")
 		(attr exclude_from_pos_files)
 		(fp_circle
@@
 		(property ki_fp_filters "Pin* Test*")
 		(sheetname "/")
-		(sheetfile "Konami Justifier 02.kicad_sch")
+		(sheetfile "Konami Justifier Main.kicad_sch")
 		(attr exclude_from_pos_files)
 		(fp_circle
@@
 		(property ki_fp_filters "Pin* Test*")
 		(sheetname "/")
-		(sheetfile "Konami Justifier 02.kicad_sch")
+		(sheetfile "Konami Justifier Main.kicad_sch")
 		(attr exclude_from_pos_files)
 		(fp_circle
@@
 		(property ki_fp_filters "Connector*:*_1x??_*")
 		(sheetname "/")
-		(sheetfile "Konami Justifier 02.kicad_sch")
+		(sheetfile "Konami Justifier Main.kicad_sch")
 		(attr through_hole)
 		(fp_line
@@
 		(property ki_fp_filters "R_*")
 		(sheetname "/")
-		(sheetfile "Konami Justifier 02.kicad_sch")
+		(sheetfile "Konami Justifier Main.kicad_sch")
 		(attr through_hole)
 		(fp_line
@@
 		(property ki_fp_filters "Connector*:*_1x??_*")
 		(sheetname "/")
-		(sheetfile "Konami Justifier 02.kicad_sch")
+		(sheetfile "Konami Justifier Main.kicad_sch")
 		(attr through_hole)
 		(fp_line
@@
 		(property ki_fp_filters "TSSOP*4.4x5mm*P0.65mm*")
 		(sheetname "/")
-		(sheetfile "Konami Justifier 02.kicad_sch")
+		(sheetfile "Konami Justifier Main.kicad_sch")
 		(attr smd)
 		(fp_line
@@
 		(property ki_fp_filters "R_*")
 		(sheetname "/")
-		(sheetfile "Konami Justifier 02.kicad_sch")
+		(sheetfile "Konami Justifier Main.kicad_sch")
 		(attr through_hole)
 		(fp_line
@@
 		(property ki_fp_filters "C_*")
 		(sheetname "/")
-		(sheetfile "Konami Justifier 02.kicad_sch")
+		(sheetfile "Konami Justifier Main.kicad_sch")
 		(attr through_hole)
 		(fp_circle
@@
 		(property ki_fp_filters "C_*")
 		(sheetname "/")
-		(sheetfile "Konami Justifier 02.kicad_sch")
+		(sheetfile "Konami Justifier Main.kicad_sch")
 		(attr through_hole)
 		(fp_line
@@
 		(property ki_fp_filters "C_*")
 		(sheetname "/")
-		(sheetfile "Konami Justifier 02.kicad_sch")
+		(sheetfile "Konami Justifier Main.kicad_sch")
 		(attr through_hole)
 		(fp_line

Commit message: Add files via upload
Parts:
- removed MD-C1: 100nF, Capacitor_THT:C_Axial_L3.8mm_D2.6mm_P10.00mm_Horizontal
- removed the SFC-C1 at (145.3, 78.5)
- added C2: 100nF, Capacitor_THT:C_Disc_D5.0mm_W2.5mm_P5.00mm, B.Cu at (150.3, 78.5)
- renumbered J3 to J2, MD-R2 to MD-R1, SFC-C2 to SFC-C1, SFC-R3 to SFC-R1
Connections:
- C1 pad 1: +5V -> GND
- C1 pad 2: GND -> +5V

Commit message: Add files via upload
Parts:
- moved C1 1.95 mm to (162.0, 109.8), turned to -90 degrees
Changed lines of the file:
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@@
 	(footprint "Capacitor_THT:C_Radial_D5.0mm_H11.0mm_P2.00mm"
 		(layer "B.Cu")
-		(at 162 111.75 90)
+		(at 162 109.8 -90)
 		(descr "C, Radial series, Radial, pin pitch=2.00mm, diameter=5mm, height=11mm, Non-Polar Electrolytic Capacitor")
 		(tags "C Radial series Radial pin pitch 2.00mm diameter 5mm height 11mm Non-Polar Electrolytic Capacitor")
 		(property "Reference" "C1"
-			(at -2.5 0 0)
+			(at 4.6 0 0)
 			(layer "B.SilkS")
 			(effects
@@
 		)
 		(pad "1" thru_hole circle
-			(at 0 0 90)
+			(at 0 0 270)
 			(size 1.6 1.6)
 			(drill 0.8)
@@
 		)
 		(pad "2" thru_hole circle
-			(at 2 0 90)
+			(at 2 0 270)
 			(size 1.6 1.6)
 			(drill 0.8)
@@
 		)
 	)
+	(gr_text "+"
+		(at 164.6 114 0)
+		(layer "B.SilkS")
+		(effects
+			(font
+				(size 1 1)
+				(thickness 0.2)
+				(bold yes)
+			)
+			(justify left bottom mirror)
+		)
+	)
 	(segment
 		(start 147.29 89.46)
@@
 	)
 	(segment
+		(start 161 117.05)
+		(end 160.4 117.65)
+		(width 1)
+		(layer "F.Cu")
+		(net 6)
+	)
+	(segment
 		(start 150.75 121.25)
 		(end 143.361 121.25)
@@
 	)
 	(segment
-		(start 161 117.05)
-		(end 160.4 117.65)
-		(width 1)
-		(layer "F.Cu")
-		(net 6)
-	)
-	(segment
 		(start 143.361 121.25)
 		(end 140.776 118.665)
@@
 	)
 	(segment
+		(start 145.3 84.4)
+		(end 145.3 81.5)
+		(width 1)
+		(layer "F.Cu")
+		(net 6)
+	)
+	(segment
+		(start 161 112.4)
+		(end 161 117.05)
+		(width 1)
+		(layer "F.Cu")
+		(net 6)
+	)
+	(segment
+		(start 158.625 106.42)
+		(end 158.625 110.025)
+		(width 1)
+		(layer "F.Cu")
+		(net 6)
+	)
+	(segment
+		(start 140.776 118.665)
+		(end 140.776 97.024)
+		(width 1)
+		(layer "F.Cu")
+		(net 6)
+	)
+	(segment
+		(start 141.31 96.49)
+		(end 141.31 88.39)
+		(width 1)
+		(layer "F.Cu")
+		(net 6)
+	)
+	(segment
+		(start 140.776 97.024)
+		(end 141.31 96.49)
+		(width 1)
+		(layer "F.Cu")
+		(net 6)
+	)
+	(segment
+		(start 145.3 81.5)
+		(end 145.3 78.54)
+		(width 1)
+		(layer "F.Cu")
+		(net 6)
+	)
+	(segment
+		(start 160.58 106.42)
+		(end 158.625 106.42)
+		(width 1)
+		(layer "F.Cu")
+		(net 6)
+	)
+	(segment
+		(start 145.3 78.54)
+		(end 145.34 78.5)
+		(width 1)
+		(layer "F.Cu")
+		(net 6)
+	)
+	(segment
+		(start 158.625 110.025)
+		(end 161 112.4)
+		(width 1)
+		(layer "F.Cu")
+		(net 6)
+	)
+	(segment
 		(start 160.4 117.65)
 		(end 150.75 117.65)
 		(width 1)
 		(layer "F.Cu")
-		(net 6)
-	)
-	(segment
-		(start 145.3 84.4)
-		(end 145.3 81.5)
-		(width 1)
-		(layer "F.Cu")
-		(net 6)
-	)
-	(segment
-		(start 161 112.75)
-		(end 161 117.05)
-		(width 1)
-		(layer "F.Cu")
-		(net 6)
-	)
-	(segment
-		(start 158.625 106.42)
-		(end 158.625 110.375)
-		(width 1)
-		(layer "F.Cu")
-		(net 6)
-	)
-	(segment
-		(start 140.776 118.665)
-		(end 140.776 97.024)
-		(width 1)
-		(layer "F.Cu")
-		(net 6)
-	)
-	(segment
-		(start 141.31 96.49)
-		(end 141.31 88.39)
-		(width 1)
-		(layer "F.Cu")
-		(net 6)
-	)
-	(segment
-		(start 140.776 97.024)
-		(end 141.31 96.49)
-		(width 1)
-		(layer "F.Cu")
-		(net 6)
-	)
-	(segment
-		(start 145.3 81.5)
-		(end 145.3 78.54)
-		(width 1)
-		(layer "F.Cu")
-		(net 6)
-	)
-	(segment
-		(start 160.58 106.42)
-		(end 158.625 106.42)
-		(width 1)
-		(layer "F.Cu")
-		(net 6)
-	)
-	(segment
-		(start 145.3 78.54)
-		(end 145.34 78.5)
-		(width 1)
-		(layer "F.Cu")
-		(net 6)
-	)
-	(segment
-		(start 158.625 110.375)
-		(end 161 112.75)
-		(width 1)
-		(layer "F.Cu")

Commit message: Add files via upload
Parts:
- J1: footprint Connector_RJ:RJ12_Amphenol_54601-x06_Horizontal -> Connector_RJ:RJ25_Wayconn_MJEA-660X1_Horizontal; moved to B.Cu
- moved J1 4.81 mm to (145.2, 119.9), turned to 180 degrees
Routing:
- net +5V: track 82.8 -> 88.6 mm
- net Net-(U1-SI): track 13.1 -> 18.1 mm
- net Net-(U1-~{CLR_LOAD}): track 10.7 -> 15.7 mm
- net Net-(U1-P/S_CONT): track 25.0 -> 27.7 mm
- net GND: track 14.7 -> 16.0 mm

Commit message: Add files via upload
Parts:
- moved C2 5.01 mm to (145.3, 78.5), turned to 0 degrees
Routing:
- net +5V: track 88.6 -> 74.3 mm
- net Net-(MD1-Pin_5): track 32.1 -> 30.9 mm

Commit message: Add files via upload
Parts:
- moved SFC-TP5 4.25 mm to (142.0, 112.5)
- moved SFC-TP6 4.20 mm to (150.8, 112.5)
- moved SFC-R1 2.84 mm to (156.8, 115.3)
- moved U1 2.80 mm to (146.7, 104.5)
- moved MD-R1 2.20 mm to (153.4, 108.9)
- moved SFC-C1 0.60 mm to (155.9, 92.1)
Routing:
- net GND: track 16.0 -> 4.42 mm
- net Net-(MD1-Pin_2): track 21.7 -> 27.3 mm
- net Net-(U1-Q/D3): track 5.16 -> 10.2 mm
- net Net-(MD1-Pin_5): track 30.9 -> 35.6 mm
- net Net-(MD1-Pin_6): track 22.4 -> 25.5 mm
- net Net-(U1-P/S_CONT): track 27.7 -> 24.9 mm
- net Net-(SFC1-Pin_2): track 21.7 -> 24.5 mm
- net Net-(MD1-Pin_1): track 22.2 -> 25.0 mm
- net Net-(J2-Pin_6): track 24.4 -> 27.2 mm
- net Net-(J2-Pin_5): track 23.4 -> 26.2 mm
- net Net-(J2-Pin_2): track 18.7 -> 21.5 mm
- net Net-(U1-~{CLR_LOAD}): track 15.7 -> 12.9 mm
- net Net-(U1-SI): track 18.1 -> 15.3 mm
- net Net-(MD1-Pin_3): track 21.6 -> 24.1 mm
- net Net-(MD1-Pin_4): track 7.21 -> 8.71 mm

Commit message: Add files via upload
Parts:
- removed SFC2: Conn_01x01_Pin, Connector_Pin:Pin_D1.0mm_L10.0mm_LooseFit
- SFC1: value Conn_01x05_Pin -> Conn_01x08_Pin; footprint Connector_Molex:Molex_SL_171971-0005_1x05_P2.54mm_Vertical -> Connector_Molex:Molex_SL_171971-0008_1x08_P2.54mm_Vertical
- moved SFC-R1 0.30 mm to (156.8, 115.0)
- moved 3.7mm 0.10 mm to (160.3, 122.2)
Other:
- outline, holes or cut-outs redrawn

Commit message: Add files via upload
Parts:
- moved 3.7mm 0.10 mm to (160.3, 122.3)
- moved J1 0.10 mm to (145.2, 119.8)
Changed lines of the file:
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@@
 		(tags "mountinghole M2 DIN965")
 		(property "Reference" "2.4mm"
-			(at -1.75 0 90)
+			(at -1.85 0 90)
 			(layer "F.SilkS")
 			(effects
@@
 	(footprint "MountingHole:MountingHole_3.7mm"
 		(layer "F.Cu")
-		(at 160.35 122.2)
+		(at 160.35 122.3)
 		(descr "Mounting Hole 3.7mm, no annular, generated by kicad-footprint-generator mountinghole.py")
 		(tags "mountinghole")
@@
 	(footprint "Connector_RJ:RJ25_Wayconn_MJEA-660X1_Horizontal"
 		(layer "B.Cu")
-		(at 145.15 119.86 180)
+		(at 145.15 119.76 180)
 		(descr "RJ25 6P6C Socket 90 degrees, https://wayconn.com/wp-content/themes/way/datasheet/MJEA-660X1XXX_RJ25_6P6C_PCB_RA.pdf")
 		(tags "RJ12 RJ18 RJ25 jack connector 6P6C")
@@
 	)
 	(zone
-		(net 4)
-		(net_name "Net-(MD1-Pin_3)")
+		(net 13)
+		(net_name "Net-(MD1-Pin_5)")
 		(layer "F.Cu")
 		(name "$teardrop_padvia$")
 		(hatch none 0.1)
-		(priority 30003)
+		(priority 30001)
 		(attr
 			(teardrop
@@
 		(polygon
 			(pts
-				(xy 160.775843 90.85) (xy 160.775843 91.65) (xy 161.146717 92.624729) (xy 162.001 92.455) (xy 162.483346 91.731621)
+				(xy 160.498612 95.930703) (xy 161.064297 96.496388) (xy 162.483346 95.718379) (xy 162.000707 94.994293)
+				(xy 161.276621 94.511654)
 			)
 		)
 	)
 	(zone
-		(net 12)
-		(net_name "Net-(MD1-Pin_6)")
+		(net 6)
+		(net_name "+5V")
 		(layer "F.Cu")
 		(name "$teardrop_padvia$")
 		(hatch none 0.1)
-		(priority 30002)
+		(priority 30000)
 		(attr
 			(teardrop
@@
 		(polygon
 			(pts
-				(xy 160.331743 98.237572) (xy 160.897428 98.803257) (xy 162.169729 98.388283) (xy 162.000707 97.534293)
-				(xy 161.276621 97.051654)
+				(xy 160.350401 105.942492) (xy 161.057508 106.649599) (xy 162.483346 105.878379) (xy 162.000707 105.154293)
+				(xy 161.276621 104.671654)
 			)
 		)
 	)
 	(zone
-		(net 6)
-		(net_name "+5V")
+		(net 12)
+		(net_name "Net-(MD1-Pin_6)")
 		(layer "F.Cu")
 		(name "$teardrop_padvia$")
 		(hatch none 0.1)
-		(priority 30000)
+		(priority 30002)
 		(attr
 			(teardrop
@@
 		(polygon
 			(pts
-				(xy 160.350401 105.942492) (xy 161.057508 106.649599) (xy 162.483346 105.878379) (xy 162.000707 105.154293)
-				(xy 161.276621 104.671654)
+				(xy 160.331743 98.237572) (xy 160.897428 98.803257) (xy 162.169729 98.388283) (xy 162.000707 97.534293)
+				(xy 161.276621 97.051654)
 			)
 		)
 	)
 	(zone
-		(net 13)
-		(net_name "Net-(MD1-Pin_5)")
+		(net 4)
+		(net_name "Net-(MD1-Pin_3)")
 		(layer "F.Cu")
 		(name "$teardrop_padvia$")
 		(hatch none 0.1)
-		(priority 30001)
+		(priority 30003)
 		(attr
 			(teardrop
@@
 		(polygon
 			(pts
-				(xy 160.498612 95.930703) (xy 161.064297 96.496388) (xy 162.483346 95.718379) (xy 162.000707 94.994293)
-				(xy 161.276621 94.511654)
+				(xy 160.775843 90.85) (xy 160.775843 91.65) (xy 161.146717 92.624729) (xy 162.001 92.455) (xy 162.483346 91.731621)
 			)
 		)
