File: Konami Justifier SFC/KiCad/Konami Justifier Main Modern/Konami Justifier Main Modern.kicad_pcb (KiCad board)
At the start: 4 copper layers, 25.2 x 50 mm, 20 parts, among them J1 RJ12, J2 Conn_01x06_Socket, U1 74VHC9164FT

Commit message: Add files via upload
Parts:
- moved SFC-TP5 1.00 mm to (142.0, 109.2)
- moved SFC-TP6 0.95 mm to (150.8, 109.2)
Routing:
- net Net-(MD1-Pin_6): track 23.0 -> 24.6 mm
- net Net-(U1-Q/D3): track 6.75 -> 5.57 mm
- net GND: track 24.9 -> 24.1 mm

Commit message: Add files via upload
Parts:
- removed SFC2: Conn_01x01_Pin, Connector_Pin:Pin_D1.0mm_L10.0mm_LooseFit
- SFC1: value Conn_01x05_Pin -> Conn_01x08_Pin; footprint Connector_Molex:Molex_SL_171971-0005_1x05_P2.54mm_Vertical -> Connector_Molex:Molex_SL_171971-0008_1x08_P2.54mm_Vertical
- moved 3.7mm 0.10 mm to (160.3, 122.2)
Other:
- board text added: "GND"
