File: Konami Justifier SFC/KiCad/Konami Justifier Main Modern/Konami Justifier Main Modern.kicad_pcb (KiCad board)
At the start: 4 copper layers, 25.2 x 50 mm, 19 parts, among them J1 RJ12, J2 Conn_01x06_Socket, U1 74VHC9164FT

Commit message: Add files via upload
Parts:
- J2: footprint Connector_Molex:Molex_SL_171971-0006_1x06_P2.54mm_Vertical -> Connector_Molex:Molex_PicoBlade_53048-0610_1x06_P1.25mm_Horizontal; moved to B.Cu
- MD1: footprint Connector_Molex:Molex_SL_171971-0009_1x09_P2.54mm_Vertical -> Connector_Molex:Molex_PicoBlade_53047-0910_1x09_P1.25mm_Vertical; moved to B.Cu
- SFC1: value Conn_01x08_Pin -> Conn_01x06_Socket; footprint Connector_Molex:Molex_SL_171971-0008_1x08_P2.54mm_Vertical -> Connector_Molex:Molex_PicoBlade_53048-0610_1x06_P1.25mm_Horizontal; moved to B.Cu
- moved J2 2.41 mm to (147.7, 81.3)
- moved SFC1 1.55 mm to (160.4, 87.3)
- moved C2 1.49 mm to (148.8, 78.6)
- moved MD1 1.29 mm to (158.3, 87.3)
- moved SFC-C1 1.17 mm to (155.9, 91.0)
- moved MD-R1 0.90 mm to (154.1, 101.8)
- moved SFC-TP1 0.20 mm to (152.8, 88.5)
- moved SFC-TP2 0.20 mm to (152.8, 91.5)
Routing:
- net +5V: track 73.8 -> 84.3 mm
- net GND: track 24.1 -> 15.4 mm, vias 4 -> 3
- net Net-(MD1-Pin_4): track 8.70 -> 13.6 mm
- net Net-(J2-Pin_6): track 24.4 -> 20.5 mm
- net Net-(MD1-Pin_3): track 20.2 -> 17.1 mm
- net Net-(MD1-Pin_6): track 24.6 -> 27.6 mm
- net Net-(J2-Pin_5): track 23.4 -> 20.7 mm
- net Net-(J2-Pin_2): track 18.7 -> 19.4 mm
- net Net-(SFC1-Pin_2): track 21.7 -> 21.9 mm, vias 0 -> 1

Commit message: Add files via upload
Parts:
- removed J2: Conn_01x06_Socket, Connector_Molex:Molex_PicoBlade_53048-0610_1x06_P1.25mm_Horizontal
- added J_BTN1: Conn_01x03, Connector_Molex:Molex_PicoBlade_53048-0310_1x03_P1.25mm_Horizontal, B.Cu at (153.8, 81.3)
- added J_IR1: Conn_01x03, Connector_Molex:Molex_PicoBlade_53048-0310_1x03_P1.25mm_Horizontal, B.Cu at (147.2, 81.3)
- moved C2 0.28 mm to (148.5, 78.6)
Routing:
- net Net-(J_BTN1-Pin_3): track 20.5 -> 23.4 mm
- net Net-(J_BTN1-Pin_2): track 20.7 -> 23.3 mm
- net +5V: track 84.3 -> 82.7 mm

Commit message: Add files via upload
Parts:
- J_BTN1, J_IR1: footprint Connector_Molex:Molex_PicoBlade_53048-0310_1x03_P1.25mm_Horizontal -> Connector_JST:JST_PH_B3B-PH-K_1x03_P2.00mm_Vertical
- MD1: footprint Connector_Molex:Molex_PicoBlade_53047-0910_1x09_P1.25mm_Vertical -> Connector_JST:JST_PH_B9B-PH-K_1x09_P2.00mm_Vertical
- SFC1: footprint Connector_Molex:Molex_PicoBlade_53048-0610_1x06_P1.25mm_Horizontal -> Connector_JST:JST_PH_B6B-PH-K_1x06_P2.00mm_Vertical
- moved J_IR1 2.51 mm to (144.9, 80.3)
- moved SFC1 1.35 mm to (161.8, 87.3)
- moved J_BTN1 1.00 mm to (153.8, 80.3)
- moved C2 0.68 mm to (147.9, 78.2)
- moved SFC-C1 0.50 mm to (155.4, 91.0)
- moved J1 0.11 mm to (145.2, 119.8)
- moved 3.7mm 0.10 mm to (160.3, 122.3)
Routing:
- net GND: track 15.4 -> 24.1 mm
- net Net-(MD1-Pin_4): track 13.6 -> 8.60 mm
- net +5V: track 82.7 -> 79.7 mm
- net Net-(MD1-Pin_6): track 27.6 -> 24.9 mm
- net Net-(MD1-Pin_3): track 17.1 -> 19.5 mm
- net Net-(MD1-Pin_5): track 33.6 -> 31.9 mm
- net Net-(J_BTN1-Pin_3): track 23.4 -> 25.1 mm
- net Net-(J_BTN1-Pin_2): track 23.3 -> 24.6 mm
- net Net-(SFC1-Pin_2): track 22.1 -> 21.9 mm, vias 1 -> 0

Commit message: Add files via upload
Parts:
- J_BTN1, J_IR1: footprint Connector_JST:JST_PH_B3B-PH-K_1x03_P2.00mm_Vertical -> Connector_Molex:Molex_PicoBlade_53048-0310_1x03_P1.25mm_Horizontal
- MD1: footprint Connector_JST:JST_PH_B9B-PH-K_1x09_P2.00mm_Vertical -> Connector_Molex:Molex_PicoBlade_53047-0910_1x09_P1.25mm_Vertical
- SFC-TP5, SFC-TP6: moved to B.Cu
- SFC1: footprint Connector_JST:JST_PH_B6B-PH-K_1x06_P2.00mm_Vertical -> Connector_Molex:Molex_PicoBlade_53047-0610_1x06_P1.25mm_Vertical
- moved SFC-TP5 6.85 mm to (142.0, 116.1), turned to 180 degrees
- moved SFC-TP6 6.85 mm to (150.8, 116.0), turned to 180 degrees
- moved C2 6.11 mm to (142.0, 79.6), turned to 90 degrees
- moved U1 6.10 mm to (146.7, 107.8)
- moved MD-R1 6.00 mm to (155.2, 95.8)
- moved SFC-R1 4.07 mm to (147.9, 117.1)
- moved J_IR1 2.65 mm to (147.4, 81.3)
- moved SFC1 1.64 mm to (162.8, 88.6)
- moved MD1 1.30 mm to (158.7, 88.6)
- moved J_BTN1 1.00 mm to (153.9, 81.3)
- moved SFC-TP1 0.70 mm to (152.1, 88.5)
- moved SFC-TP2 0.70 mm to (152.1, 91.5)
- moved SFC-TP3 0.55 mm to (141.7, 88.5)
- moved SFC-TP4 0.55 mm to (141.7, 91.5)
- moved SFC-C1 0.37 mm to (155.3, 90.7)
Routing:
- net Net-(U1-Q/D3): track 5.57 -> 16.2 mm
- net Net-(SFC1-Pin_2): track 21.9 -> 31.6 mm
- net Net-(MD1-Pin_6): track 24.9 -> 33.6 mm
- net Net-(MD1-Pin_3): track 19.5 -> 27.6 mm
- net Net-(MD1-Pin_1): track 22.1 -> 29.6 mm
- net Net-(MD1-Pin_2): track 21.5 -> 27.7 mm
- net Net-(U1-~{CLR_LOAD}): track 15.7 -> 9.55 mm
- net Net-(U1-SI): track 18.1 -> 12.0 mm
- net Net-(U1-P/S_CONT): track 27.7 -> 21.6 mm
- net Net-(J_IR1-Pin_2): track 19.5 -> 25.3 mm
- net GND: track 24.1 -> 18.3 mm
- net Net-(J_BTN1-Pin_2): track 24.6 -> 30.0 mm
- net Net-(J_BTN1-Pin_3): track 25.1 -> 30.1 mm
- net Net-(MD1-Pin_4): track 8.60 -> 4.56 mm
- net Net-(MD1-Pin_5): track 31.9 -> 35.7 mm
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Other:
- board text added: "+5v"
- board text added: "CLK"
- board text added: "DA1"
- board text added: "PIO"
- board text added: "STR"
