File: Konami Justifier SFC/KiCad/Konami Justifier Main Modern/Konami Justifier Main Modern.kicad_sch (KiCad schematic)
At the start: 17 parts, among them J1 RJ12, J2 Conn_01x06_Socket, U1 74VHC9164FT

Commit message: Add files via upload
Parts:
- removed SFC1: Conn_01x05_Pin, Connector_Molex:Molex_SL_171971-0005_1x05_P2.54mm_Vertical, symbol Connector:Conn_01x05_Pin
- removed SFC2: Conn_01x01_Pin, Connector_Pin:Pin_D1.0mm_L10.0mm_LooseFit, symbol Connector:Conn_01x01_Pin
- added SFC1: Conn_01x08_Pin, Connector_Molex:Molex_SL_171971-0008_1x08_P2.54mm_Vertical, symbol Connector:Conn_01x08_Pin
Connections:
- net +5V: now also SFC1.8 (Pin_8)
- net GND: now also SFC1.1 (Pin_1)
- net at SFC-TP1.1, U1.10 (Q/D5): now also SFC1.2 (Pin_2)
- net at MD1.3 (Pin_3), SFC-C1.1, U1.9 (Q/D4): now also SFC1.3 (Pin_3)
- net at MD1.5 (Pin_5), SFC-TP2.1, U1.5 (Q/D1): now also SFC1.4 (Pin_4)
- net at MD1.6 (Pin_6), SFC-TP6.1, U1.6 (Q/D2): now also SFC1.5 (Pin_5)
- no-connect marks 0 -> 2
Changed lines of the file:
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@@
 		(color 0 0 0 0)
 	)
+	(no_connect
+		(at 161.29 59.69)
+	)
+	(no_connect
+		(at 161.29 57.15)
+	)
 	(wire
 		(pts
@@
 	(wire
 		(pts
+			(xy 161.29 54.61) (xy 187.96 54.61)
+		)
+		(stroke
+			(width 0)
+			(type default)
+		)
+	)
+	(wire
+		(pts
 			(xy 153.67 74.93) (xy 153.67 121.92)
 		)
@@
 	(wire
 		(pts
-			(xy 179.07 63.5) (xy 184.15 63.5)
+			(xy 161.29 44.45) (xy 177.8 44.45)
 		)
 		(stroke
@@
 	(wire
 		(pts
-			(xy 187.96 54.61) (xy 177.8 54.61)
+			(xy 161.29 52.07) (xy 196.85 52.07)
 		)
 		(stroke
@@
 	(wire
 		(pts
-			(xy 190.5 46.99) (xy 177.8 46.99)
-		)
-		(stroke
-			(width 0)
-			(type default)
-		)
-	)
-	(wire
-		(pts
 			(xy 95.25 134.62) (xy 86.36 134.62)
 		)
@@
 	(wire
 		(pts
+			(xy 161.29 63.5) (xy 161.29 62.23)
+		)
+		(stroke
+			(width 0)
+			(type default)
+		)
+	)
+	(wire
+		(pts
 			(xy 95.25 127) (xy 85.09 127)
 		)
@@
 	(wire
 		(pts
+			(xy 161.29 63.5) (xy 184.15 63.5)
+		)
+		(stroke
+			(width 0)
+			(type default)
+		)
+	)
+	(wire
+		(pts
 			(xy 151.13 74.93) (xy 151.13 95.25)
 		)
@@
 	(wire
 		(pts
+			(xy 161.29 46.99) (xy 190.5 46.99)
+		)
+		(stroke
+			(width 0)
+			(type default)
+		)
+	)
+	(wire
+		(pts
 			(xy 69.85 62.23) (xy 69.85 64.77)
 		)
@@
 	(wire
 		(pts
-			(xy 193.04 49.53) (xy 177.8 49.53)
-		)
-		(stroke
-			(width 0)
-			(type default)
-		)
-	)
-	(wire
-		(pts
 			(xy 187.96 124.46) (xy 187.96 54.61)
 		)
@@
 	(wire
 		(pts
+			(xy 161.29 49.53) (xy 193.04 49.53)
+		)
+		(stroke
+			(width 0)
+			(type default)
+		)
+	)
+	(wire
+		(pts
 			(xy 156.21 74.93) (xy 156.21 124.46)
 		)
@@
 		(pts
 			(xy 95.25 129.54) (xy 88.9 129.54)
-		)
-		(stroke
-			(width 0)
-			(type default)
-		)
-	)
-	(wire
-		(pts
-			(xy 177.8 52.07) (xy 196.85 52.07)
 		)
 		(stroke
@@
 	)
 	(symbol
-		(lib_id "Connector:Conn_01x05_Pin")
-		(at 172.72 49.53 0)
-		(unit 1)
-		(exclude_from_sim no)
-		(in_bom yes)
-		(on_board yes)
-		(dnp no)
-		(fields_autoplaced yes)
-		(property "Reference" "SFC1"
-			(at 173.355 39.37 0)
-			(effects
-				(font
-					(size 1.27 1.27)
-				)
-			)
-		)
-		(property "Value" "Conn_01x05_Pin"
-			(at 173.355 41.91 0)
-			(effects
-				(font
-					(size 1.27 1.27)
-				)
-			)
-		)
-		(property "Footprint" "Connector_Molex:Molex_SL_171971-0005_1x05_P2.54mm_Vertical"
-			(at 172.72 49.53 0)
-			(effects
-				(font
-					(size 1.27 1.27)
-				)
-				(hide yes)
-			)
-		)
-		(property "Datasheet" "~"
-			(at 172.72 49.53 0)
-			(effects
-				(font
-					(size 1.27 1.27)
-				)
-				(hide yes)
-			)
-		)
-		(property "Description" "Generic connector, single row, 01x05, script generated"
-			(at 172.72 49.53 0)
-			(effects
-				(font
-					(size 1.27 1.27)
-				)
-				(hide yes)
-			)
-		)
-		(pin "2"
-		)
-		(pin "5"
-		)
-		(pin "1"
-		)
-		(pin "3"
-		)
-		(pin "4"
-		)
-		(instances
-			(project ""
-				(path "/57790297-21ee-4532-bd10-fc40752b9a93"
-					(reference "SFC1")
-					(unit 1)
-				)
-			)
-		)
-	)
-	(symbol
 		(lib_id "power:+5V")
 		(at 220.98 93.98 0)
@@
 	)
 	(symbol
-		(lib_id "Connector:Conn_01x01_Pin")
-		(at 173.99 63.5 0)
-		(unit 1)
-		(exclude_from_sim no)
-		(in_bom yes)
-		(on_board yes)
-		(dnp no)
-		(fields_autoplaced yes)
-		(property "Reference" "SFC2"
-			(at 174.625 58.42 0)
-			(effects
-				(font
-					(size 1.27 1.27)
-				)
-			)
-		)
-		(property "Value" "Conn_01x01_Pin"
-			(at 174.625 60.96 0)
-			(effects
-				(font
-					(size 1.27 1.27)
-				)
-			)
-		)
-		(property "Footprint" "Connector_Pin:Pin_D1.0mm_L10.0mm_LooseFit"
-			(at 173.99 63.5 0)
-			(effects
-				(font
-					(size 1.27 1.27)
-				)
-				(hide yes)
-			)
-		)
-		(property "Datasheet" "~"
-			(at 173.99 63.5 0)
-			(effects
-				(font
-					(size 1.27 1.27)
-				)
-				(hide yes)
-			)
-		)
-		(property "Description" "Generic connector, single row, 01x01, script generated"
-			(at 173.99 63.5 0)
-			(effects
-				(font
-					(size 1.27 1.27)
-				)
-				(hide yes)
-			)
-		)
-		(pin "1"
-		)
-		(instances
-			(project ""
-				(path "/57790297-21ee-4532-bd10-fc40752b9a93"
-					(reference "SFC2")
-					(unit 1)
-				)
-			)
-		)
-	)
-	(symbol
 		(lib_id "power:GND")
 		(at 95.25 158.75 0)
@@
 					(unit 1)
 				)
+			)
+		)
+	)
+	(symbol
+		(lib_id "Connector:Conn_01x08_Pin")
+		(at 156.21 52.07 0)
+		(unit 1)
+		(exclude_from_sim no)
+		(in_bom yes)
+		(on_board yes)
+		(dnp no)
+		(fields_autoplaced yes)
+		(property "Reference" "SFC1"
+			(at 156.845 39.37 0)
+			(effects
+				(font
+					(size 1.27 1.27)
+				)
+			)
+		)
+		(property "Value" "Conn_01x08_Pin"
+			(at 156.845 41.91 0)
+			(effects
+				(font
+					(size 1.27 1.27)
+				)
+			)
+		)
+		(property "Footprint" "Connector_Molex:Molex_SL_171971-0008_1x08_P2.54mm_Vertical"
+			(at 156.21 52.07 0)
+			(effects
+				(font
+					(size 1.27 1.27)
+				)
+				(hide yes)
+			)
+		)
+		(property "Datasheet" "~"
+			(at 156.21 52.07 0)
+			(effects
+				(font
+					(size 1.27 1.27)
+				)
+				(hide yes)
+			)
+		)
+		(property "Description" "Generic connector, single row, 01x08, script generated"
+			(at 156.21 52.07 0)
+			(effects
+				(font
+					(size 1.27 1.27)
+				)
+				(hide yes)
+			)
+		)
+		(pin "3"
+		)
+		(pin "1"
+		)
+		(pin "7"
+		)
+		(pin "2"
+		)
+		(pin "4"
+		)
+		(pin "6"
+		)
+		(pin "8"
+		)
+		(pin "5"
+		)
+		(instances
+			(project ""
+				(path "/57790297-21ee-4532-bd10-fc40752b9a93"
+					(reference "SFC1")
+					(unit 1)
+				)

Commit message: Add files via upload
Parts:
- removed SFC1: Conn_01x08_Pin, Connector_Molex:Molex_SL_171971-0008_1x08_P2.54mm_Vertical, symbol Connector:Conn_01x08_Pin
- added SFC1: Conn_01x06_Socket, Connector_Molex:Molex_PicoBlade_53048-0610_1x06_P1.25mm_Horizontal, symbol Connector:Conn_01x06_Socket
- J2: footprint Connector_Molex:Molex_SL_171971-0006_1x06_P2.54mm_Vertical -> Connector_Molex:Molex_PicoBlade_53048-0610_1x06_P1.25mm_Horizontal
- MD1: footprint Connector_Molex:Molex_SL_171971-0009_1x09_P2.54mm_Vertical -> Connector_Molex:Molex_PicoBlade_53047-0910_1x09_P1.25mm_Vertical
Connections:
- net +5V: now also SFC1.6 (Pin_6)
- net GND: now also SFC1.1 (Pin_1)
- net at MD1.3 (Pin_3), SFC-C1.1, U1.9 (Q/D4): now also SFC1.3 (Pin_3)
- net at SFC-TP1.1, U1.10 (Q/D5): now also SFC1.2 (Pin_2)
- net at MD1.5 (Pin_5), SFC-TP2.1, U1.5 (Q/D1): now also SFC1.4 (Pin_4)
- net at MD1.6 (Pin_6), SFC-TP6.1, U1.6 (Q/D2): now also SFC1.5 (Pin_5)
- no-connect marks 2 -> 0
Changed lines of the file:
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@@
 		(color 0 0 0 0)
 	)
-	(no_connect
-		(at 161.29 59.69)
-	)
-	(no_connect
-		(at 161.29 57.15)
-	)
 	(wire
 		(pts
@@
 	(wire
 		(pts
-			(xy 161.29 63.5) (xy 161.29 62.23)
-		)
-		(stroke
-			(width 0)
-			(type default)
-		)
-	)
-	(wire
-		(pts
 			(xy 95.25 127) (xy 85.09 127)
 		)
@@
 		(pts
 			(xy 167.64 119.38) (xy 167.64 124.46)
+		)
+		(stroke
+			(width 0)
+			(type default)
+		)
+	)
+	(wire
+		(pts
+			(xy 161.29 57.15) (xy 161.29 63.5)
 		)
 		(stroke
@@
 			)
 		)
-		(property "Footprint" "Connector_Molex:Molex_SL_171971-0006_1x06_P2.54mm_Vertical"
+		(property "Footprint" "Connector_Molex:Molex_PicoBlade_53048-0610_1x06_P1.25mm_Horizontal"
 			(at 69.85 57.15 0)
 			(effects
@@
 	)
 	(symbol
+		(lib_id "Connector:Conn_01x06_Socket")
+		(at 156.21 49.53 0)
+		(mirror y)
+		(unit 1)
+		(exclude_from_sim no)
+		(in_bom yes)
+		(on_board yes)
+		(dnp no)
+		(fields_autoplaced yes)
+		(property "Reference" "SFC1"
+			(at 156.845 39.37 0)
+			(effects
+				(font
+					(size 1.27 1.27)
+				)
+			)
+		)
+		(property "Value" "Conn_01x06_Socket"
+			(at 156.845 41.91 0)
+			(effects
+				(font
+					(size 1.27 1.27)
+				)
+			)
+		)
+		(property "Footprint" "Connector_Molex:Molex_PicoBlade_53048-0610_1x06_P1.25mm_Horizontal"
+			(at 156.21 49.53 0)
+			(effects
+				(font
+					(size 1.27 1.27)
+				)
+				(hide yes)
+			)
+		)
+		(property "Datasheet" "~"
+			(at 156.21 49.53 0)
+			(effects
+				(font
+					(size 1.27 1.27)
+				)
+				(hide yes)
+			)
+		)
+		(property "Description" "Generic connector, single row, 01x06, script generated"
+			(at 156.21 49.53 0)
+			(effects
+				(font
+					(size 1.27 1.27)
+				)
+				(hide yes)
+			)
+		)
+		(pin "3"
+		)
+		(pin "2"
+		)
+		(pin "4"
+		)
+		(pin "1"
+		)
+		(pin "6"
+		)
+		(pin "5"
+		)
+		(instances
+			(project ""
+				(path "/57790297-21ee-4532-bd10-fc40752b9a93"
+					(reference "SFC1")
+					(unit 1)
+				)
+			)
+		)
+	)
+	(symbol
 		(lib_id "Connector:TestPoint_Alt")
 		(at 196.85 71.12 270)
@@
 	)
 	(symbol
-		(lib_id "Connector:Conn_01x08_Pin")
-		(at 156.21 52.07 0)
-		(unit 1)
-		(exclude_from_sim no)
-		(in_bom yes)
-		(on_board yes)
-		(dnp no)
-		(fields_autoplaced yes)
-		(property "Reference" "SFC1"
-			(at 156.845 39.37 0)
-			(effects
-				(font
-					(size 1.27 1.27)
-				)
-			)
-		)
-		(property "Value" "Conn_01x08_Pin"
-			(at 156.845 41.91 0)
-			(effects
-				(font
-					(size 1.27 1.27)
-				)
-			)
-		)
-		(property "Footprint" "Connector_Molex:Molex_SL_171971-0008_1x08_P2.54mm_Vertical"
-			(at 156.21 52.07 0)
-			(effects
-				(font
-					(size 1.27 1.27)
-				)
-				(hide yes)
-			)
-		)
-		(property "Datasheet" "~"
-			(at 156.21 52.07 0)
-			(effects
-				(font
-					(size 1.27 1.27)
-				)
-				(hide yes)
-			)
-		)
-		(property "Description" "Generic connector, single row, 01x08, script generated"
-			(at 156.21 52.07 0)
-			(effects
-				(font
-					(size 1.27 1.27)
-				)
-				(hide yes)
-			)
-		)
-		(pin "3"
-		)
-		(pin "1"
-		)
-		(pin "7"
-		)
-		(pin "2"
-		)
-		(pin "4"
-		)
-		(pin "6"
-		)
-		(pin "8"
-		)
-		(pin "5"
-		)
-		(instances
-			(project ""
-				(path "/57790297-21ee-4532-bd10-fc40752b9a93"
-					(reference "SFC1")
-					(unit 1)
-				)
-			)
-		)
-	)
-	(symbol
 		(lib_id "74xx:74VHC9164FT")
 		(at 107.95 132.08 0)
@@
 			)
 		)
-		(property "Footprint" "Connector_Molex:Molex_SL_171971-0009_1x09_P2.54mm_Vertical"
+		(property "Footprint" "Connector_Molex:Molex_PicoBlade_53047-0910_1x09_P1.25mm_Vertical"
 			(at 153.67 69.85 0)
 			(effects

Commit message: Add files via upload
Parts:
- removed J2: Conn_01x06_Socket, Connector_Molex:Molex_PicoBlade_53048-0610_1x06_P1.25mm_Horizontal, symbol Connector:Conn_01x06_Socket
- added J_BTN1, J_IR1: Conn_01x03, Connector_Molex:Molex_PicoBlade_53048-0310_1x03_P1.25mm_Horizontal, symbol Connector_Generic:Conn_01x03
Connections:
- net +5V: now also J_IR1.1 (Pin_1)
- net GND: now also J_BTN1.1 (Pin_1), J_IR1.3 (Pin_3)
- net at U1.15 (Q8C): now also J_IR1.2 (Pin_2)
- net at U1.14 (Q8'): now also J_BTN1.2 (Pin_2)
- net at U1.13 (Q/D8): now also J_BTN1.3 (Pin_3)

Commit message: Add files via upload
Parts:
- J_BTN1, J_IR1: footprint Connector_Molex:Molex_PicoBlade_53048-0310_1x03_P1.25mm_Horizontal -> Connector_JST:JST_PH_B3B-PH-K_1x03_P2.00mm_Vertical
- MD1: footprint Connector_Molex:Molex_PicoBlade_53047-0910_1x09_P1.25mm_Vertical -> Connector_JST:JST_PH_B9B-PH-K_1x09_P2.00mm_Vertical
- SFC1: footprint Connector_Molex:Molex_PicoBlade_53048-0610_1x06_P1.25mm_Horizontal -> Connector_JST:JST_PH_B6B-PH-K_1x06_P2.00mm_Vertical
Changed lines of the file:
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@@
 			)
 		)
-		(property "Footprint" "Connector_Molex:Molex_PicoBlade_53048-0310_1x03_P1.25mm_Horizontal"
+		(property "Footprint" "Connector_JST:JST_PH_B3B-PH-K_1x03_P2.00mm_Vertical"
 			(at 60.96 38.1 0)
 			(effects
@@
 			)
 		)
-		(property "Footprint" "Connector_Molex:Molex_PicoBlade_53048-0310_1x03_P1.25mm_Horizontal"
+		(property "Footprint" "Connector_JST:JST_PH_B3B-PH-K_1x03_P2.00mm_Vertical"
 			(at 78.74 38.1 0)
 			(effects
@@
 			)
 		)
-		(property "Footprint" "Connector_Molex:Molex_PicoBlade_53048-0610_1x06_P1.25mm_Horizontal"
+		(property "Footprint" "Connector_JST:JST_PH_B6B-PH-K_1x06_P2.00mm_Vertical"
 			(at 156.21 49.53 0)
 			(effects
@@
 			)
 		)
-		(property "Footprint" "Connector_Molex:Molex_PicoBlade_53047-0910_1x09_P1.25mm_Vertical"
+		(property "Footprint" "Connector_JST:JST_PH_B9B-PH-K_1x09_P2.00mm_Vertical"
 			(at 153.67 69.85 0)
 			(effects

Commit message: Add files via upload
Parts:
- J_BTN1, J_IR1: footprint Connector_JST:JST_PH_B3B-PH-K_1x03_P2.00mm_Vertical -> Connector_Molex:Molex_PicoBlade_53048-0310_1x03_P1.25mm_Horizontal
- MD1: footprint Connector_JST:JST_PH_B9B-PH-K_1x09_P2.00mm_Vertical -> Connector_Molex:Molex_PicoBlade_53047-0910_1x09_P1.25mm_Vertical
- SFC1: footprint Connector_JST:JST_PH_B6B-PH-K_1x06_P2.00mm_Vertical -> Connector_Molex:Molex_PicoBlade_53047-0610_1x06_P1.25mm_Vertical
Changed lines of the file:
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@@
 			)
 		)
-		(property "Footprint" "Connector_JST:JST_PH_B3B-PH-K_1x03_P2.00mm_Vertical"
+		(property "Footprint" "Connector_Molex:Molex_PicoBlade_53048-0310_1x03_P1.25mm_Horizontal"
 			(at 60.96 38.1 0)
 			(effects
@@
 			)
 		)
-		(property "Footprint" "Connector_JST:JST_PH_B3B-PH-K_1x03_P2.00mm_Vertical"
+		(property "Footprint" "Connector_Molex:Molex_PicoBlade_53048-0310_1x03_P1.25mm_Horizontal"
 			(at 78.74 38.1 0)
 			(effects
@@
 			)
 		)
-		(property "Footprint" "Connector_JST:JST_PH_B6B-PH-K_1x06_P2.00mm_Vertical"
+		(property "Footprint" "Connector_Molex:Molex_PicoBlade_53047-0610_1x06_P1.25mm_Vertical"
 			(at 156.21 49.53 0)
 			(effects
@@
 			)
 		)
-		(property "Footprint" "Connector_JST:JST_PH_B9B-PH-K_1x09_P2.00mm_Vertical"
+		(property "Footprint" "Connector_Molex:Molex_PicoBlade_53047-0910_1x09_P1.25mm_Vertical"
 			(at 153.67 69.85 0)
 			(effects
