File: Konami Justifier SFC/KiCad/Konami Justifier Start/Konami Justifier Start.kicad_pcb (KiCad board)
At the start: 4 copper layers, 15.2 x 15.4 mm, 7 parts, among them SW1 SW_Push_Open

Commit message: Add files via upload
Parts:
- moved TP1 0.17 mm to (141.8, 105.4)
- moved TP2 0.11 mm to (146.0, 105.4)
Changed lines of the file:
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@@
 	(footprint "TestPoint:TestPoint_THTPad_D1.5mm_Drill0.7mm"
 		(layer "F.Cu")
-		(at 141.63 105.4)
+		(at 141.8 105.4)
 		(descr "THT pad as test Point, diameter 1.5mm, hole diameter 0.7mm")
 		(tags "test point THT pad")
@@
 		(pad "" np_thru_hole circle
 			(at 0 0 90)
-			(size 5.3 5.3)
-			(drill 5.3)
+			(size 4.8 4.8)
+			(drill 4.8)
 			(layers "*.Cu" "*.Mask")
 		)
@@
 	(footprint "TestPoint:TestPoint_THTPad_D1.5mm_Drill0.7mm"
 		(layer "F.Cu")
-		(at 146.11 105.4)
+		(at 146 105.4)
 		(descr "THT pad as test Point, diameter 1.5mm, hole diameter 0.7mm")
 		(tags "test point THT pad")
@@
 			(fill no)
 			(layer "Cmts.User")
-			(net 7798903)
 		)
 		(fp_circle
@@
 			(fill no)
 			(layer "F.CrtYd")
-			(net 7798903)
 		)
 		(pad "" np_thru_hole circle
@@
 		(pad "" np_thru_hole circle
 			(at 0 0 270)
-			(size 5.3 5.3)
-			(drill 5.3)
+			(size 4.8 4.8)
+			(drill 4.8)
 			(layers "*.Cu" "*.Mask")
 		)

Commit message: Add files via upload
Parts:
- moved REF** 0.10 mm to (151.4, 99.2)
- moved REF** 0.10 mm to (136.3, 99.2)
Changed lines of the file:
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@@
 		(tenting front back)
 		(pcbplotparams
-			(layerselection 0x00000000_00000000_55555555_5755f5ff)
+			(layerselection 0x00000000_00000000_55555555_5755f5af)
 			(plot_on_all_layers_selection 0x00000000_00000000_00000000_00000000)
 			(disableapertmacros no)
@@
 			(outputformat 1)
 			(mirror no)
-			(drillshape 1)
+			(drillshape 0)
 			(scaleselection 1)
-			(outputdirectory "")
+			(outputdirectory "C:/Users/ifreund/Documents/Konami Justifier Start/Gerbers/")
 		)
 	)
@@
 		(locked yes)
 		(layer "F.Cu")
-		(at 151.5 99.199838 90)
+		(at 151.4 99.199838 90)
 		(descr "Mounting Hole 5.3mm, M5, no annular, generated by kicad-footprint-generator mountinghole.py")
 		(tags "mountinghole M5")
@@
 		(locked yes)
 		(layer "F.Cu")
-		(at 136.25 99.2 -90)
+		(at 136.35 99.2 -90)
 		(descr "Mounting Hole 5.3mm, M5, no annular, generated by kicad-footprint-generator mountinghole.py")
 		(tags "mountinghole M5")
@@
 	)
 	(gr_text "GND"
-		(at 138.5 105.75 90)
+		(at 138.925 106.15 90)
 		(layer "F.Cu" knockout)
 		(effects
 			(font
-				(size 1 1)
-				(thickness 0.2)
+				(size 1.25 1.25)
+				(thickness 0.25)
 				(bold yes)
 			)
