File: Konami Justifier SFC/KiCad/Konami Justifier Top/Konami Justifier Top.kicad_pcb (KiCad board)
At the start: 4 copper layers, 15.2 x 50 mm, 10 parts, among them J1 RJ12, U1 IS485

Commit message: Add files via upload
Parts:
- moved ? 0.60 mm to (152.2, 86.2)
- moved REF** 0.60 mm to (142.6, 86.2)
- moved ? 0.20 mm to (147.4, 80.6)
Changed lines of the file:
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@@
 	(footprint ""
 		(layer "F.Cu")
-		(at 147.4 80.4 90)
+		(at 147.4 80.6 90)
 		(property "Reference" ""
 			(at 0 0 90)
@@
 	(footprint ""
 		(layer "F.Cu")
-		(at 152.2 85.6)
+		(at 152.2 86.2)
 		(property "Reference" ""
 			(at 0 0 0)
@@
 	(footprint "MountingHole:MountingHole_2.2mm_M2_DIN965_Pad"
 		(layer "F.Cu")
-		(at 142.6 85.6)
+		(at 142.6 86.2)
 		(descr "Mounting Hole 2.2mm, M2, generated by kicad-footprint-generator mountinghole.py")
 		(tags "mountinghole M2 DIN965")

Commit message: Add files via upload
Parts:
- C1, R1: moved to B.Cu
Routing:
- net GND: track 40.4 -> 30.9 mm
Other:
- board text added: "GND"

Commit message: Add files via upload
Routing:
- net GND: track 30.9 -> 21.4 mm
Changed lines of the file:
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@@
 	)
 	(segment
-		(start 144 96.5)
-		(end 144 95.8)
-		(width 0.25)
+		(start 148.75 113)
+		(end 148.75 101.25)
+		(width 0.4)
 		(layer "F.Cu")
 		(net 1)
 	)
 	(segment
-		(start 148.75 113)
-		(end 148.75 108)
-		(width 0.25)
+		(start 148.75 101.25)
+		(end 144 96.5)
+		(width 0.4)
 		(layer "F.Cu")
 		(net 1)
@@
 		(start 144 95.8)
 		(end 145.4 94.4)
-		(width 0.25)
+		(width 0.4)
 		(layer "F.Cu")
 		(net 1)
 	)
 	(segment
-		(start 148.75 108)
-		(end 148.75 101.25)
-		(width 0.25)
-		(layer "F.Cu")
-		(net 1)
-	)
-	(segment
-		(start 148.75 101.25)
-		(end 144 96.5)
-		(width 0.25)
+		(start 144 96.5)
+		(end 144 95.8)
+		(width 0.4)
 		(layer "F.Cu")
 		(net 1)
@@
 		(start 142 101.5)
 		(end 142 101.25)
-		(width 0.25)
-		(layer "F.Cu")
-		(net 1)
-	)
-	(segment
-		(start 142 101.25)
-		(end 148.75 108)
 		(width 0.25)
 		(layer "F.Cu")
@@
 	)
 	(segment
-		(start 153 94.535)
-		(end 148.8 90.335)
-		(width 0.5)
+		(start 151.9 109.7)
+		(end 153 108.6)
+		(width 1)
 		(layer "F.Cu")
 		(net 2)
 	)
 	(segment
-		(start 151.8 112.95)
-		(end 151.8 109.8)
-		(width 0.5)
+		(start 149.2 84.66)
+		(end 148.8 84.26)
+		(width 1)
 		(layer "F.Cu")
 		(net 2)
@@
 	(segment
 		(start 153 108.6)
-		(end 153 94.535)
-		(width 0.5)
+		(end 153 94)
+		(width 1)
 		(layer "F.Cu")
 		(net 2)
 	)
 	(segment
-		(start 148.8 90.335)
-		(end 148.8 84.26)
-		(width 0.5)
+		(start 151.9 113.4)
+		(end 151.9 109.7)
+		(width 1)
 		(layer "F.Cu")
 		(net 2)
 	)
 	(segment
-		(start 151.8 109.8)
-		(end 153 108.6)
-		(width 0.5)
+		(start 149.2 90.2)
+		(end 149.2 84.66)
+		(width 1)
+		(layer "F.Cu")
+		(net 2)
+	)
+	(segment
+		(start 153 94)
+		(end 149.2 90.2)
+		(width 1)
 		(layer "F.Cu")
 		(net 2)
@@
 		(start 147.6 98.43)
 		(end 147.6 85.6)
-		(width 0.25)
+		(width 0.4)
 		(layer "F.Cu")
 		(net 4)
@@
 		(start 150.25 115)
 		(end 150.25 101.08)
-		(width 0.25)
+		(width 0.4)
 		(layer "F.Cu")
 		(net 4)
@@
 		(start 150.25 101.08)
 		(end 147.6 98.43)
-		(width 0.25)
+		(width 0.4)
 		(layer "F.Cu")
 		(net 4)
@@
 	(segment
 		(start 142 109.25)
-		(end 144.25 111.5)
-		(width 0.25)
+		(end 144.4 111.65)
+		(width 0.4)
 		(layer "F.Cu")
 		(net 5)
 	)
 	(segment
-		(start 144.25 111.5)
-		(end 144.25 115)
-		(width 0.25)
+		(start 144.4 111.65)
+		(end 144.4 115.4)
+		(width 0.4)
 		(layer "F.Cu")
 		(net 5)
 	)
 	(segment
-		(start 145.75 109)
-		(end 142 105.25)
-		(width 0.25)
+		(start 145.9 113.4)
+		(end 145.9 109.15)
+		(width 0.4)
 		(layer "F.Cu")
 		(net 6)
 	)
 	(segment
-		(start 145.75 113)
-		(end 145.75 109)
-		(width 0.25)
+		(start 145.9 109.15)
+		(end 142 105.25)
+		(width 0.4)
 		(layer "F.Cu")
 		(net 6)

Commit message: Add files via upload
Parts:
- J1: footprint Connector_JST:JST_ZE_B06B-ZESK-D_1x06_P1.50mm_Vertical -> Connector_RJ:RJ25_Wayconn_MJEA-660X1_Horizontal
- moved J1 2.22 mm to (149.9, 114.5), turned to 0 degrees
Routing:
- net Net-(U1-OUT): track 31.2 -> 33.5 mm
- net Net-(J1-Pad6): track 7.14 -> 9.08 mm
- net GND: track 21.4 -> 22.7 mm
- net Net-(J1-Pad5): track 9.77 -> 11.0 mm
- net +5V: track 31.5 -> 30.5 mm
