File: Konami Justifier SFC/KiCad/Konami Justifier Main JST-PH/Konami Justifier Main JST-PH.kicad_pcb (KiCad board)
At the start: 4 copper layers, 25.2 x 50 mm, 19 parts, among them J1 RJ12, J2 Conn_01x06, U1 74VHC9164FT

Commit message: Add files via upload
Parts:
- moved SFC-TP5 0.65 mm to (142.0, 115.1)
- moved SFC-TP6 0.65 mm to (150.8, 115.0)
- moved J2 0.30 mm to (156.9, 79.6)
Routing:
- net GND: track 20.2 -> 23.8 mm
